File: receiver/receiver.kicad_sch (KiCad schematic)
At the start: 19 parts, among them Q1 BC327, Q2 BC337, Q3 IRF804, Q4 IRF804, Q5 BC337, Q6 BC327, Q7 IRF804, Q8 BC337, Q9 BC327

Commit message: new schematic
Parts:
- added C1, C2, C3: 4.7uF, symbol Device:C_Polarized_Small
Connections:
- net +5V: now also C1.1; no longer D2.1 (K), D3.1 (K), Q5.1 (C), Q8.1 (C)
- net GND: now also C1.2, C2.2, C3.2
- new net Motor1+: C3.1, D3.1 (K), Q8.1 (C)
- new net Motor2+: C2.1, D2.1 (K), Q5.1 (C)
Other:
- moved on the sheet: D1, Q1, Q2, Q3, R1
